Commit message: update urdf

File: prbt_cell_description/urdf/workcell.urdf (robot description, URDF)
Before this commit: robot prbt_workcell, 8 links, 7 joints
Links:
- added link prbt_base
- added link prbt_base_link, mass 2.4; collision cylinder length=0.13 radius=0.09275; visual mesh filename=package://prbt_robot_support/meshes/foot.dae
- added link prbt_flange, mass 0.02; collision cylinder length=0.02 radius=0.0331; visual mesh filename=package://prbt_robot_support/meshes/flange.dae
- added link prbt_link_1, mass 7.1; collision cylinder length=0.10 radius=0.065; collision cylinder length=0.10 radius=0.07
- added link prbt_link_2, mass 1.7; collision box size=0.11 0.1 0.075; collision box size=0.121 0.27 0.065
- added link prbt_link_3, mass 4.8; collision cylinder length=0.10 radius=0.06; collision cylinder length=0.10 radius=0.065
- added link prbt_link_4, mass 0.9; collision box size=0.09 0.06 0.12; collision box size=0.121 0.08 0.17
- added link prbt_link_5, mass 2.6; collision cylinder length=0.03 radius=0.05; collision cylinder length=0.04 radius=0.0545
- added link prbt_tool0
Joints:
- added joint prbt__robot_cell_joint: type fixed, parent robot_link, child prbt_base_link
- added joint prbt_base_link-base: type fixed, parent prbt_base_link, child prbt_base, origin xyz=0 0 0 rpy=0 0 0
- added joint prbt_flange-tool0: type fixed, parent prbt_flange, child prbt_tool0, origin xyz=0 0 0 rpy=0 0 0
- added joint prbt_joint_1: type revolute, parent prbt_base_link, child prbt_link_1, origin xyz=0 0 0.2604 rpy=0 0 -3.141592653589793, axis 0 0 1, limit lower=-2.96706 upper=2.96706 effort=370 velocity=1.57
- added joint prbt_joint_2: type revolute, parent prbt_link_1, child prbt_link_2, origin xyz=0 0 0 rpy=1.5707963267948966 0 0, axis 0 0 1, limit lower=-2.53073 upper=2.53073 effort=370 velocity=1.57
- added joint prbt_joint_3: type revolute, parent prbt_link_2, child prbt_link_3, origin xyz=0 0.35 0 rpy=0 3.141592653589793 0, axis 0 0 1, limit lower=-2.35620 upper=2.35620 effort=176 velocity=1.57
- added joint prbt_joint_4: type revolute, parent prbt_link_3, child prbt_link_4, origin xyz=0 0 0 rpy=-1.5707963267948966 3.141592653589793 0, axis 0 0 1, limit lower=-2.96706 upper=2.96706 effort=176 velocity=1.57
- added joint prbt_joint_5: type revolute, parent prbt_link_4, child prbt_link_5, origin xyz=0 0 0.307 rpy=1.5707963267948966 0 3.141592653589793, axis 0 0 1, limit lower=-2.96706 upper=2.96706 effort=41.6 velocity=1.57
- added joint prbt_joint_6: type revolute, parent prbt_link_5, child prbt_flange, origin xyz=0 0.084 0 rpy=-1.5707963267948966 0 0, axis 0 0 1, limit lower=-3.12414 upper=3.12414 effort=20.1 velocity=1.57
