Commit message: Update workcell with prbt robot.

File: prbt_cell_description/urdf/workcell.urdf.xacro (robot description, xacro)
@@ -1,5 +1,7 @@
 <?xml version="1.0"?>
 <robot xmlns:xacro="http://www.ros.org/wiki/xacro" name="prbt_workcell">
+    <xacro:arg name="robot_prefix" default="prbt_"/>
     <xacro:include filename="$(find prbt_cell_description)/urdf/robot_cell.xacro"/>
+    <xacro:include filename="$(find prbt_robot_support)/urdf/prbt_macro.xacro" />
     <!-- Add world link -->
     <link name="world" />
@@ -7,3 +9,9 @@
         <origin xyz="0 0 0" rpy="0 0 0" />
     </xacro:robot_cell>
+    <!-- Add robot -->
+    <xacro:prbt prefix="$(arg robot_prefix)" />
+    <joint name="$(arg robot_prefix)_robot_cell_joint" type="fixed">
+        <parent link="robot_link"/>
+        <child link="$(arg robot_prefix)base_link"/>
+    </joint>
 </robot>

Commit message: update meshes

File: prbt_cell_description/urdf/workcell.urdf.xacro (robot description, xacro)
@@ -3,4 +3,5 @@
     <xacro:arg name="robot_prefix" default="prbt_"/>
     <xacro:include filename="$(find prbt_cell_description)/urdf/robot_cell.xacro"/>
+    <xacro:include filename="$(find prbt_cell_description)/urdf/schunk_egp40.xacro" />
     <xacro:include filename="$(find prbt_robot_support)/urdf/prbt_macro.xacro" />
     <!-- Add world link -->
@@ -15,3 +16,7 @@
         <child link="$(arg robot_prefix)base_link"/>
     </joint>
+    <!-- Add gripper -->
+    <xacro:schunk_egp40 name="gripper" prefix="$(arg robot_prefix)" parent="$(arg robot_prefix)tool0">
+        <origin xyz="0 0 0" rpy="0 0 0" />
+    </xacro:schunk_egp40>
 </robot>

Commit message: Include realsense camera

File: prbt_cell_description/urdf/workcell.urdf.xacro (robot description, xacro)
@@ -2,7 +2,11 @@
 <robot xmlns:xacro="http://www.ros.org/wiki/xacro" name="prbt_workcell">
     <xacro:arg name="robot_prefix" default="prbt_"/>
+    <xacro:arg name="use_nominal_extrinsics" default="false"/>
+    <xacro:arg name="add_plug" default="false" />
+    <xacro:arg name="use_mesh" default="true" />
     <xacro:include filename="$(find prbt_cell_description)/urdf/robot_cell.xacro"/>
     <xacro:include filename="$(find prbt_cell_description)/urdf/schunk_egp40.xacro" />
     <xacro:include filename="$(find prbt_robot_support)/urdf/prbt_macro.xacro" />
+    <xacro:include filename="$(find realsense2_description)/urdf/_d435.urdf.xacro" />
     <!-- Add world link -->
     <link name="world" />
@@ -20,3 +24,7 @@
         <origin xyz="0 0 0" rpy="0 0 0" />
     </xacro:schunk_egp40>
+    <!-- Add camera -->
+    <xacro:sensor_d435 parent="$(arg robot_prefix)schunk_egp40_base_link" use_nominal_extrinsics="$(arg use_nominal_extrinsics)" add_plug="$(arg add_plug)" use_mesh="$(arg use_mesh)">
+        <origin xyz="0 -0.05 ${0.015+0.010}" rpy="0 -${pi/2} ${pi/2}"/>
+    </xacro:sensor_d435>
 </robot>
