Commit message: Complete gripper with flange

File: prbt_cell_description/urdf/schunk_egp40.xacro (robot description, xacro)
@@ -1,4 +1,4 @@
 <?xml version="1.0"?>
-<robot xmlns:xacro="http://www.ros.org/wiki/xacro" name="schunk_egp50">
+<robot xmlns:xacro="http://www.ros.org/wiki/xacro" name="schunk_egp40">
     <xacro:macro name="schunk_egp40" params="
         name
@@ -8,6 +8,6 @@
     ">
         <xacro:include filename="inertial_macros.xacro" />
-        <xacro:property name="base_diameter" value="0.075" />
-        <xacro:property name="base_length" value="0.015" />
+        <xacro:property name="base_diameter" value="0.065" />
+        <xacro:property name="base_height" value="0.015" />
         <xacro:property name="body_length" value="0.04" />
         <xacro:property name="body_width" value="0.026" />
@@ -27,27 +27,24 @@
         </material>
         <!--Base plate-->
-        <link name="${prefix}schunk_egp50_base_link">
+        <link name="${prefix}schunk_egp40_base_link">
             <visual>
                 <geometry>
-                    <cylinder length="${base_length}" radius="${base_diameter/2}" />
+                    <mesh filename="package://prbt_cell_description/meshes/flange_v3.STL" scale="0.001 0.001 0.001" />
                 </geometry>
                 <material name="blue" />
-                <origin rpy="0 0 0" xyz="0 0 ${base_length/2}" />
+                <origin rpy="${pi} 0 0" xyz="-${base_diameter/2} ${base_diameter/2} ${base_height}" />
             </visual>
             <collision>
                 <geometry>
-                    <cylinder length="${base_length}" radius="${base_diameter/2}" />
+                    <mesh filename="package://prbt_cell_description/meshes/flange_v3.STL" scale="0.001 0.001 0.001" />
                 </geometry>
-                <origin rpy="0 0 0" xyz="0 0 ${base_length/2}" />
+                <origin rpy="${pi} 0 0" xyz="-${base_diameter/2} ${base_diameter/2} ${base_height}" />
             </collision>
-            <xacro:inertial_cylinder mass="0.2" length="${base_length}" radius="${base_diameter/2}">
-                <origin rpy="0 0 0" xyz="0 0 ${base_length/2}" />
-            </xacro:inertial_cylinder>
         </link>
         <!--Main gripper-->
-        <link name="${prefix}schunk_egp50_body_link">
+        <link name="${prefix}schunk_egp40_body_link">
             <visual>
                 <geometry>
-                    <mesh filename="package://prbt_cell_description/meshes/Gripper.stl" scale="0.001 0.001 0.001" />
+                    <mesh filename="package://prbt_cell_description/meshes/schunk_egp40_body.STL" scale="0.001 0.001 0.001" />
                 </geometry>
                 <origin rpy="${pi/2} 0 0" xyz="${-body_length/2} ${body_width/2} ${-body_height/2}" />
@@ -56,5 +53,5 @@
             <collision>
                 <geometry>
-                    <mesh filename="package://prbt_cell_description/meshes/Gripper.stl" scale="0.001 0.001 0.001" />
+                    <mesh filename="package://prbt_cell_description/meshes/schunk_egp40_body.STL" scale="0.001 0.001 0.001" />
                 </geometry>
                 <origin rpy="${pi/2} 0 0" xyz="${-body_length/2} ${body_width/2} ${-body_height/2}" />
@@ -65,8 +62,8 @@
         </link>
         <!--Pincer block 1-->
-        <link name="${prefix}schunk_egp50_pincer_1_link">
+        <link name="${prefix}schunk_egp40_finger_left_link">
             <visual>
                 <geometry>
-                    <mesh filename="package://prbt_cell_description/meshes/Pincer_1.stl" scale="0.001 0.001 0.001" />
+                    <mesh filename="package://prbt_cell_description/meshes/schunk_finger_left.STL" scale="0.001 0.001 0.001" />
                 </geometry>
                 <origin rpy="${pi/2} 0 0" xyz="${-body_length/2} ${pincer_width/2} ${-body_height-pincer_height/2}" />
@@ -75,5 +72,5 @@
             <collision>
                 <geometry>
-                    <mesh filename="package://prbt_cell_description/meshes/Pincer_1.stl" scale="0.001 0.001 0.001" />
+                    <mesh filename="package://prbt_cell_description/meshes/schunk_finger_left.STL" scale="0.001 0.001 0.001" />
                 </geometry>
                 <origin rpy="${pi/2} 0 0" xyz="${-body_length/2} ${pincer_width/2} ${-body_height-pincer_height/2}" />
@@ -84,8 +81,8 @@
         </link>
         <!--Pincer block 2-->
-        <link name="${prefix}schunk_egp50_pincer_2_link">
+        <link name="${prefix}schunk_egp40_finger_right_link">
             <visual>
                 <geometry>
-                    <mesh filename="package://prbt_cell_description/meshes/Pincer_2.stl" scale="0.001 0.001 0.001" />
+                    <mesh filename="package://prbt_cell_description/meshes/schunk_finger_right.STL" scale="0.001 0.001 0.001" />
                 </geometry>
                 <origin rpy="${pi/2} 0 0" xyz="${-body_length/2} ${pincer_width/2} ${-body_height-pincer_height/2}" />
@@ -94,5 +91,5 @@
             <collision>
                 <geometry>
-                    <mesh filename="package://prbt_cell_description/meshes/Pincer_2.stl" scale="0.001 0.001 0.001" />
+                    <mesh filename="package://prbt_cell_description/meshes/schunk_finger_right.STL" scale="0.001 0.001 0.001" />
                 </geometry>
                 <origin rpy="${pi/2} 0 0" xyz="${-body_length/2} ${pincer_width/2} ${-body_height-pincer_height/2}" />
@@ -105,12 +102,12 @@
         <link name="tool_tip" />
         <!-- Joints-->
-        <joint name="${prefix}schunk_egp50_body_joint" type="fixed">
-            <parent link="${prefix}schunk_egp50_base_link" />
-            <child link="${prefix}schunk_egp50_body_link" />
-            <origin xyz="0.0 0.0 ${base_length+body_height/2}" rpy="0.0 0.0 0.0" />
+        <joint name="${prefix}schunk_egp40_body_joint" type="fixed">
+            <parent link="${prefix}schunk_egp40_base_link" />
+            <child link="${prefix}schunk_egp40_body_link" />
+            <origin xyz="0.0 0.0 ${body_height/2+base_height}" rpy="0.0 0.0 0.0" />
         </joint>
-        <joint name="${prefix}schunk_egp50_pincer_1_joint" type="fixed">
-            <parent link="${prefix}schunk_egp50_body_link" />
-            <child link="${prefix}schunk_egp50_pincer_1_link" />
+        <joint name="${prefix}schunk_egp40_finger_left_joint" type="fixed">
+            <parent link="${prefix}schunk_egp40_body_link" />
+            <child link="${prefix}schunk_egp40_finger_left_link" />
             <origin xyz="0.0 0.0 ${body_height/2+pincer_height/2}" rpy="0.0 0.0 0.0" />
             <!-- the motion of the pincer is along the X axis -->
@@ -119,7 +116,7 @@
             <limit lower="${-body_length/16}" upper="${body_length/16}" velocity="100" effort="100" />
         </joint>
-        <joint name="schunk_egp50_pincer_2_joint" type="fixed">
-            <parent link="${prefix}schunk_egp50_body_link" />
-            <child link="${prefix}schunk_egp50_pincer_2_link" />
+        <joint name="schunk_egp40_finger_right_joint" type="fixed">
+            <parent link="${prefix}schunk_egp40_body_link" />
+            <child link="${prefix}schunk_egp40_finger_right_link" />
             <origin xyz="0.0 0.002 ${body_height/2+pincer_height/2}" rpy="0.0 0.0 0.0" />
             <!-- the motion of the pincer is along the X axis -->
@@ -128,15 +125,15 @@
             <limit lower="${body_length/16}" upper="${-body_length/16}" velocity="100" effort="100" />
         </joint>
-        <joint name="${prefix}schunk_egp50_tip_joint" type="fixed">
-            <parent link="${prefix}schunk_egp50_base_link" />
+        <joint name="${prefix}schunk_egp40_tip_joint" type="fixed">
+            <parent link="${prefix}schunk_egp40_base_link" />
             <child link="tool_tip" />
             <origin xyz="0 0 ${body_height_max}" rpy="0.0 0.0 0.0" />
         </joint>
         <joint
-            name="schunk_egp50_base_joint"
+            name="schunk_egp40_base_joint"
             type="fixed"
         >
             <parent link="${parent}" />
-            <child link="${prefix}schunk_egp50_base_link" />
+            <child link="${prefix}schunk_egp40_base_link" />
             <xacro:insert_block name="origin" />
         </joint>

Commit message: update flange

File: prbt_cell_description/urdf/schunk_egp40.xacro (robot description, xacro)
@@ -30,5 +30,5 @@
             <visual>
                 <geometry>
-                    <mesh filename="package://prbt_cell_description/meshes/flange_v3.STL" scale="0.001 0.001 0.001" />
+                    <mesh filename="package://prbt_cell_description/meshes/flange_v2.6.STL" scale="0.001 0.001 0.001" />
                 </geometry>
                 <material name="blue" />
@@ -37,5 +37,5 @@
             <collision>
                 <geometry>
-                    <mesh filename="package://prbt_cell_description/meshes/flange_v3.STL" scale="0.001 0.001 0.001" />
+                    <mesh filename="package://prbt_cell_description/meshes/flange_v2.6.STL" scale="0.001 0.001 0.001" />
                 </geometry>
                 <origin rpy="${pi} 0 0" xyz="-${base_diameter/2} ${base_diameter/2} ${base_height}" />

Commit message: update flange model

File: prbt_cell_description/urdf/schunk_egp40.xacro (robot description, xacro)
@@ -30,5 +30,5 @@
             <visual>
                 <geometry>
-                    <mesh filename="package://prbt_cell_description/meshes/flange_v2.6.STL" scale="0.001 0.001 0.001" />
+                    <mesh filename="package://prbt_cell_description/meshes/flange_v3.STL" scale="0.001 0.001 0.001" />
                 </geometry>
                 <material name="blue" />
@@ -37,5 +37,5 @@
             <collision>
                 <geometry>
-                    <mesh filename="package://prbt_cell_description/meshes/flange_v2.6.STL" scale="0.001 0.001 0.001" />
+                    <mesh filename="package://prbt_cell_description/meshes/flange_v3.STL" scale="0.001 0.001 0.001" />
                 </geometry>
                 <origin rpy="${pi} 0 0" xyz="-${base_diameter/2} ${base_diameter/2} ${base_height}" />
