Commit message: remove ros2 components

File: prbt_cell_description/urdf/prbt_cell.urdf.xacro (robot description, xacro)
@@ -2,8 +2,4 @@
 <robot xmlns:xacro="http://www.ros.org/wiki/xacro" name="prbt_cell">
     <xacro:arg name="robot_prefix" default="prbt_"/>
-    <xacro:arg name="bus_config" default="$(find prbt_robot_support)/config/prbt/bus.yml"/>
-    <xacro:arg name="master_config" default="$(find prbt_robot_support)/config/prbt/master.dcf"/>
-    <xacro:arg name="can_interface_name" default="vcan0"/>
-    <xacro:arg name="master_bin" default=""/>
     <xacro:arg name="use_nominal_extrinsics" default="false"/>
     <xacro:arg name="add_plug" default="false" />
@@ -11,6 +7,5 @@
     <xacro:include filename="$(find prbt_cell_description)/urdf/robot_cell.xacro"/>
     <xacro:include filename="$(find prbt_cell_description)/urdf/schunk_egp40.xacro" />
-    <xacro:include filename="$(find prbt_robot_support)/urdf/prbt_macro.xacro" />
-    <xacro:include filename="$(find prbt_robot_support)/urdf/prbt.ros2_control.xacro" />
+    <xacro:include filename="$(find prbt_support)/urdf/prbt_macro.xacro" />
     <xacro:include filename="$(find realsense2_description)/urdf/_d435.urdf.xacro" />
     <!-- Add world link -->
@@ -20,14 +15,10 @@
     </xacro:robot_cell>
     <!-- Add robot -->
-    <xacro:prbt prefix="$(arg robot_prefix)" parent="robot_link">
-        <origin xyz="0 0 0" rpy="0 0 -${pi/2}" />
-    </xacro:prbt>
-    <xacro:prbt_ros2_control
-        name="$(arg robot_prefix)"
-        prefix="$(arg robot_prefix)"
-        bus_config="$(arg bus_config)"
-        master_config="$(arg master_config)"
-        can_interface_name="$(arg can_interface_name)"
-        master_bin="$(arg master_bin)" />
+    <xacro:prbt prefix="$(arg robot_prefix)" />
+    <joint name="$(arg robot_prefix)base_link_cell_joint" type="fixed">
+      <origin xyz="0 0 0" rpy="0 0 -${pi/2}" />
+      <parent link="robot_link"/>
+      <child link="$(arg robot_prefix)base_link"/>
+    </joint>
     <!-- Add gripper -->
     <xacro:schunk_egp40 name="gripper" prefix="" parent="$(arg robot_prefix)tool0">

Commit message: calibration data

File: prbt_cell_description/urdf/prbt_cell.urdf.xacro (robot description, xacro)
@@ -28,4 +28,5 @@
     <xacro:sensor_d435 parent="schunk_egp40_base_link" use_nominal_extrinsics="$(arg use_nominal_extrinsics)" add_plug="$(arg add_plug)" use_mesh="$(arg use_mesh)">
         <origin xyz="0 -0.05 ${0.015+0.010}" rpy="0 -${pi/2} ${pi/2}"/>
+        <!-- <origin xyz="-0.091 0.0069 -0.1782" rpy="3.1307 0.1792 0.1233" /> -->
     </xacro:sensor_d435>
 </robot>
