Commit message: final calibration

File: prbt_cell_description/urdf/prbt_cell.urdf (robot description, URDF)
Before this commit: robot prbt_cell, 24 links, 23 joints
Joints:
- joint camera_joint: origin xyz=0 -0.05 0.025 rpy=0 -1.5707963267948966 1.5707963267948966 -> xyz=-0.0130762 -0.0636807 0.0292817 rpy=1.52494 -0.0110301 1.57125; parent schunk_egp40_base_link -> prbt_tool0
- joint schunk_egp40_finger_left_joint: type prismatic -> fixed
- joint schunk_egp40_finger_right_joint: type prismatic -> fixed

File: prbt_cell_description/urdf/schunk_egp40.xacro (robot description, xacro)
@@ -107,5 +107,5 @@
             <origin xyz="0.0 0.0 ${body_height/2+base_height}" rpy="0.0 0.0 0.0" />
         </joint>
-        <joint name="${prefix}schunk_egp40_finger_left_joint" type="prismatic">
+        <joint name="${prefix}schunk_egp40_finger_left_joint" type="fixed">
             <parent link="${prefix}schunk_egp40_body_link" />
             <child link="${prefix}schunk_egp40_finger_left_link" />
@@ -116,5 +116,5 @@
             <limit lower="${-body_length/16}" upper="${body_length/16}" velocity="100" effort="100" />
         </joint>
-        <joint name="schunk_egp40_finger_right_joint" type="prismatic">
+        <joint name="schunk_egp40_finger_right_joint" type="fixed">
             <parent link="${prefix}schunk_egp40_body_link" />
             <child link="${prefix}schunk_egp40_finger_right_link" />
