Commit message: testing new robot cell

File: prbt_cell_description/urdf/robot_cell.xacro (robot description, xacro)
@@ -20,5 +20,5 @@
             <visual>
                 <geometry>
-                    <mesh filename="package://prbt_cell_description/meshes/Assembly_new.STL" scale="0.001 0.001 0.001" />
+                    <mesh filename="package://prbt_cell_description/meshes/prbt_cell_v1.0.STL" scale="0.001 0.001 0.001" />
                 </geometry>
                 <material name="gray"/>

File: prbt_cell_description/urdf/workcell.urdf.xacro (robot description, xacro)
@@ -20,5 +20,5 @@
     </xacro:robot_cell>
     <!-- Add robot -->
-    <xacro:prbt prefix="$(arg robot_prefix)" />
+    <!-- <xacro:prbt prefix="$(arg robot_prefix)" />
     <joint name="$(arg robot_prefix)_robot_cell_joint" type="fixed">
         <parent link="robot_link"/>
@@ -31,12 +31,12 @@
         master_config="$(arg master_config)"
         can_interface_name="$(arg can_interface_name)"
-        master_bin="$(arg master_bin)" />
+        master_bin="$(arg master_bin)" /> -->
     <!-- Add gripper -->
-    <xacro:schunk_egp40 name="gripper" prefix="$(arg robot_prefix)" parent="$(arg robot_prefix)tool0">
+    <!-- <xacro:schunk_egp40 name="gripper" prefix="$(arg robot_prefix)" parent="$(arg robot_prefix)tool0">
         <origin xyz="0 0 0" rpy="0 0 0" />
-    </xacro:schunk_egp40>
+    </xacro:schunk_egp40> -->
     <!-- Add camera -->
-    <xacro:sensor_d435 parent="$(arg robot_prefix)schunk_egp40_base_link" use_nominal_extrinsics="$(arg use_nominal_extrinsics)" add_plug="$(arg add_plug)" use_mesh="$(arg use_mesh)">
+    <!-- <xacro:sensor_d435 parent="$(arg robot_prefix)schunk_egp40_base_link" use_nominal_extrinsics="$(arg use_nominal_extrinsics)" add_plug="$(arg add_plug)" use_mesh="$(arg use_mesh)">
         <origin xyz="0 -0.05 ${0.015+0.010}" rpy="0 -${pi/2} ${pi/2}"/>
-    </xacro:sensor_d435>
+    </xacro:sensor_d435> -->
 </robot>

Commit message: New robot cell position correction

File: prbt_cell_description/urdf/robot_cell.xacro (robot description, xacro)
@@ -7,11 +7,11 @@
         parent
         *origin">
-        <xacro:property name="robot_center_offset_length" value="0.42" />
+        <xacro:property name="robot_center_offset_length" value="0.315" />
         <xacro:property name="robot_center_offset_width" value="0.02" />
-        <xacro:property name="robot_base_height" value="0.99" />
-        <xacro:property name="robotcell_length" value="1.44" />
-        <xacro:property name="robotcell_width" value="0.94" />
+        <xacro:property name="robot_base_height" value="0.62" />
+        <xacro:property name="robotcell_length" value="1.20" />
+        <xacro:property name="robotcell_width" value="0.80" />
         <xacro:property name="robotcell_height" value="1.16" />
-        <xacro:property name="shield_thickness" value="0.03" />
+        <xacro:property name="shield_thickness" value="0.045" />
         <material name="gray">
             <color rgba="0.6 0.8 0.8 1" />
@@ -41,9 +41,9 @@
                 <origin rpy="0 0 0 " xyz="0 0 0" />
                 <geometry>
-                    <box size="${robotcell_length} ${shield_thickness} ${robotcell_height}" />
+                    <box size="${robotcell_length} ${shield_thickness*2} ${robotcell_height}" />
                 </geometry>
                 <material name="gray"/>
             </collision>
-            <xacro:inertial_box mass="5" x="${robotcell_length}" y="${shield_thickness}" z="${robotcell_height}">
+            <xacro:inertial_box mass="5" x="${robotcell_length}" y="${shield_thickness*2}" z="${robotcell_height}">
                 <origin rpy="0 0 0" xyz="0 0 0" />
             </xacro:inertial_box>
@@ -89,5 +89,5 @@
             <parent link="${prefix}robotcell_base_link" />
             <child link="${prefix}visuals_link" />
-            <origin xyz="${robotcell_length/2+shield_thickness} -${robotcell_width/2+shield_thickness} 0" rpy="0 0 ${pi/2}" />
+            <origin xyz="${robotcell_length/2} -${robotcell_width/2} 0" rpy="0 0 ${pi/2}" />
         </joint>
         <joint name="${prefix}robotcell_base_to_front_joint" type="fixed">
@@ -99,5 +99,5 @@
             <parent link="${prefix}robotcell_base_link" />
             <child link="${prefix}shield_rear_link" />
-            <origin xyz="0 ${-robotcell_width/2+shield_thickness/2} ${robot_base_height+robotcell_height/2}" rpy="0 0 0" />
+            <origin xyz="0 ${-robotcell_width/2+shield_thickness} ${robot_base_height+robotcell_height/2}" rpy="0 0 0" />
         </joint>
         <joint name="${prefix}robotcell_base_to_left" type="fixed">

File: prbt_cell_description/urdf/workcell.urdf (robot description, URDF)
Before this commit: robot prbt_workcell, 17 links, 16 joints
Links:
- link robotcell_base_link: geometry collision box size=1.2 0.8 0.62
- link shield_front_link: geometry collision box size=1.2 0.045 1.16
- link shield_left_link: geometry collision box size=0.045 0.8 1.16
- link shield_rear_link: geometry collision box size=1.2 0.09 1.16
- link shield_right_link: geometry collision box size=0.045 0.8 1.16
- link visuals_link: geometry visual mesh filename=package://prbt_cell_description/meshes/prbt_cell_v1.0.STL scale=0.001 0.001 0.001
Joints:
- removed joint prbt__robot_cell_joint
- added joint prbt_base_link_robot_link_joint: type fixed, parent robot_link, child prbt_base_link, origin xyz=0 0 0 rpy=0 0 0
- joint robot_cell_base_to_robot_link: origin xyz=0.42 0.02 0.99 rpy=0 0 0 -> xyz=0.315 0.0 0.62 rpy=0 0 0
- joint robotcell_base_to_front_joint: origin xyz=0 0.45499999999999996 1.5699999999999998 rpy=0 0 0 -> xyz=0 0.3775 1.2 rpy=0 0 0
- joint robotcell_base_to_left: origin xyz=-0.705 0 1.5699999999999998 rpy=0 0 0 -> xyz=-0.5775 0 1.2 rpy=0 0 0
- joint robotcell_base_to_rear: origin xyz=0 -0.45499999999999996 1.5699999999999998 rpy=0 0 0 -> xyz=0 -0.35500000000000004 1.2 rpy=0 0 0
- joint robotcell_base_to_right: origin xyz=0.705 0 1.5699999999999998 rpy=0 0 0 -> xyz=0.5775 0 1.2 rpy=0 0 0
- joint robotcell_base_to_visual: origin xyz=0.75 -0.5 0 rpy=0 0 1.5707963267948966 -> xyz=0.6 -0.4 0 rpy=0 0 1.5707963267948966

File: prbt_cell_description/urdf/workcell.urdf.xacro (robot description, xacro)
@@ -20,9 +20,7 @@
     </xacro:robot_cell>
     <!-- Add robot -->
-    <!-- <xacro:prbt prefix="$(arg robot_prefix)" />
-    <joint name="$(arg robot_prefix)_robot_cell_joint" type="fixed">
-        <parent link="robot_link"/>
-        <child link="$(arg robot_prefix)base_link"/>
-    </joint>
+    <xacro:prbt prefix="$(arg robot_prefix)" parent="robot_link">
+        <origin xyz="0 0 0" rpy="0 0 -${pi/2}" />
+    </xacro:prbt>
     <xacro:prbt_ros2_control
         name="$(arg robot_prefix)"
@@ -31,12 +29,12 @@
         master_config="$(arg master_config)"
         can_interface_name="$(arg can_interface_name)"
-        master_bin="$(arg master_bin)" /> -->
+        master_bin="$(arg master_bin)" />
     <!-- Add gripper -->
-    <!-- <xacro:schunk_egp40 name="gripper" prefix="$(arg robot_prefix)" parent="$(arg robot_prefix)tool0">
+    <xacro:schunk_egp40 name="gripper" prefix="$(arg robot_prefix)" parent="$(arg robot_prefix)tool0">
         <origin xyz="0 0 0" rpy="0 0 0" />
-    </xacro:schunk_egp40> -->
+    </xacro:schunk_egp40>
     <!-- Add camera -->
-    <!-- <xacro:sensor_d435 parent="$(arg robot_prefix)schunk_egp40_base_link" use_nominal_extrinsics="$(arg use_nominal_extrinsics)" add_plug="$(arg add_plug)" use_mesh="$(arg use_mesh)">
+    <xacro:sensor_d435 parent="$(arg robot_prefix)schunk_egp40_base_link" use_nominal_extrinsics="$(arg use_nominal_extrinsics)" add_plug="$(arg add_plug)" use_mesh="$(arg use_mesh)">
         <origin xyz="0 -0.05 ${0.015+0.010}" rpy="0 -${pi/2} ${pi/2}"/>
-    </xacro:sensor_d435> -->
+    </xacro:sensor_d435>
 </robot>

Commit message: include base plate collision

File: prbt_cell_description/urdf/robot_cell.xacro (robot description, xacro)
@@ -85,4 +85,16 @@
             </xacro:inertial_box>
         </link>
+        <link name="${prefix}robotcell_collision_base_link">
+            <collision>
+                <origin rpy="0 0 0" xyz="0 0 ${robot_base_height/2}" />
+                <geometry>
+                    <box size="${robotcell_length} ${robotcell_width} ${robot_base_height+0.12}" />
+                </geometry>
+                <material name="gray"/>
+            </collision>
+            <xacro:inertial_box mass="70" x="${robotcell_length}" y="${robotcell_width}" z="${robot_base_height+0.12}">
+                <origin rpy="0 0 0" xyz="0 0 0" />
+            </xacro:inertial_box>
+        </link>
         <link name="${prefix}robot_link" />
         <joint name="${prefix}robotcell_base_to_visual" type="fixed">
@@ -116,4 +128,9 @@
             <xacro:insert_block name="origin" />
         </joint>
+        <joint name="${prefix}robot_cell_collision_base_joint" type="fixed">
+            <parent link="${parent}" />
+            <child link="${prefix}robotcell_collision_base_link" />
+            <xacro:insert_block name="origin" />
+        </joint>
         <joint name="${prefix}robot_cell_base_to_robot_link" type="fixed">
             <parent link="${prefix}robotcell_base_link" />

Commit message: include collision object

File: prbt_cell_description/urdf/robot_cell.xacro (robot description, xacro)
@@ -97,4 +97,16 @@
             </xacro:inertial_box>
         </link>
+        <link name="${prefix}robotcell_collision_object_link">
+            <collision>
+                <origin rpy="0 0 0" xyz="0 0 0" />
+                <geometry>
+                    <box size="0.1 0.6 0.15" />
+                </geometry>
+                <material name="gray"/>
+            </collision>
+            <xacro:inertial_box mass="70" x="${robotcell_length}" y="${robotcell_width}" z="${robot_base_height+0.12}">
+                <origin rpy="0 0 0" xyz="0 0 0" />
+            </xacro:inertial_box>
+        </link>
         <link name="${prefix}robot_link" />
         <joint name="${prefix}robotcell_base_to_visual" type="fixed">
@@ -138,4 +150,9 @@
             <origin xyz="${robot_center_offset_length} ${robot_center_offset_width} ${robot_base_height}" rpy="0 0 0" />
         </joint>
+        <joint name="${prefix}robot_cell_collision_object_link" type="fixed">
+            <parent link="${prefix}robot_link" />
+            <child link="${prefix}robotcell_collision_object_link" />
+            <origin xyz="-0.25 0 0.2" rpy="0 0 0" />
+        </joint>
     </xacro:macro>
 </robot>
